File: CPUs/pepper/pepper-8m/pepper-8m.sch (EAGLE design)
At the start: 22 parts

Commit message: this is version 0.2
the board is only 0.1" shorter and the silscreeen was corected in oreder
o add part numbers
Parts:
- XT1: device abracon-resonators:AWSCR-12.00MGD-C -> abracon-resonators:AWSCR-12.00CR-C; EAGLEUP CERAMIC740X340-3N -> (none)
Other:
- note added: "www.hotboards.org"
- note removed: "admin@stackblocks.org"
- note removed: "www.stackblocks.org"
Changed lines of the file:
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@@
 <?xml version="1.0" encoding="utf-8"?>
 <!DOCTYPE eagle SYSTEM "eagle.dtd">
-<eagle version="6.2">
+<eagle version="6.4">
 <drawing>
 <settings>
@@
 <setting verticaltext="up"/>
 </settings>
-<grid distance="0.1" unitdist="inch" unit="inch" style="lines" multiple="1" display="yes" altdistance="0.01" altunitdist="inch" altunit="inch"/>
+<grid distance="0.1" unitdist="inch" unit="inch" style="lines" multiple="1" display="no" altdistance="0.01" altunitdist="inch" altunit="inch"/>
 <layers>
 <layer number="1" name="Top" color="4" fill="1" visible="no" active="no"/>
@@
 <part name="SW1" library="esw-tactile-sw" deviceset="TL3301?*J" device="N" technology="F160Q"/>
 <part name="SW2" library="esw-tactile-sw" deviceset="TL3301?*J" device="N" technology="F160Q"/>
-<part name="XT1" library="abracon-resonators" deviceset="AWSCR-*MGD-C" device="" technology="12.00" value="12MHz">
-<attribute name="EAGLEUP" value="CERAMIC740X340-3N"/>
-</part>
 <part name="IC1" library="st-ldos" deviceset="LD1117?*" device="S" technology="33TR">
 <attribute name="EAGLEUP" value="SOT230P700X180-4N"/>
@@
 <part name="R3" library="te-fixed-resistors" deviceset="CRG?*" device="0603" technology="F390R" value="390"/>
 <part name="R4" library="te-fixed-resistors" deviceset="CRG?*" device="0603" technology="F390R" value="390"/>
+<part name="XT1" library="abracon-resonators" deviceset="AWSCR-*CR-C" device="" technology="12.00" value="12MHz"/>
 </parts>
 <sheets>
@@
 <text x="45.72" y="180.34" size="2.54" layer="97">Coupling Capacitors </text>
 <text x="238.76" y="7.62" size="2.54" layer="94">1.0</text>
-<text x="187.96" y="45.72" size="3.81" layer="98">www.stackblocks.org</text>
-<text x="180.34" y="38.1" size="3.81" layer="98">admin@stackblocks.org</text>
 <text x="149.86" y="25.4" size="2.54" layer="94">for pic18f microcontrollers</text>
 <text x="5.08" y="7.62" size="1.778" layer="98" ratio="12">Not populated</text>
@@
 <text x="124.46" y="43.18" size="1.778" layer="98" ratio="12">Not populated</text>
 <text x="81.28" y="132.08" size="2.54" layer="97" ratio="12">Power Led</text>
+<wire x1="124.46" y1="106.68" x2="177.8" y2="106.68" width="0.3048" layer="98"/>
+<text x="193.04" y="38.1" size="3.81" layer="98">www.hotboards.org</text>
 </plain>
 <instances>
@@
 <instance part="SW1" gate="G$1" x="10.16" y="104.14"/>
 <instance part="SW2" gate="G$1" x="48.26" y="101.6"/>
-<instance part="XT1" gate="G$1" x="12.7" y="63.5" rot="R270"/>
 <instance part="IC1" gate="G$1" x="20.32" y="160.02"/>
 <instance part="IC2" gate="G$1" x="132.08" y="149.86"/>
@@
 <instance part="R3" gate="G$1" x="68.58" y="111.76" rot="R90"/>
 <instance part="R4" gate="G$1" x="91.44" y="116.84" rot="R90"/>
+<instance part="XT1" gate="G$1" x="12.7" y="63.5" rot="R270"/>
 </instances>
 <busses>
